Commit message: feat: SLAM pronto - TF tree completa e LiDAR funcional
- LiDAR publicando a 25Hz no tópico /scan
- TF tree: odom -> base_link -> lidarA2
- Bridge Gazebo-Harmonic configurado
- Nó tf_remapper para correção de frames
- Ackermann steering controller configurado
- Mundo museum.world com sensores ativos

Próximo passo: Configurar SLAM Toolbox

File: src/camaro_description/urdf/camaro.xacro (robot description, xacro)
@@ -167,5 +167,5 @@
     <limit lower="-1.79769e+308" upper="1.79769e+308" effort="100" velocity="100"/>
   </joint>
-  <!-- ========== SENSOR LIDAR ========== -->
+  <!-- ========== SENSOR LIDAR (CORRIGIDO: SEM COLISÃO) ========== -->
   <link name="lidarA2">
     <inertial>
@@ -178,7 +178,4 @@
       <material name="red"><color rgba="1 0 0 1"/></material>
     </visual>
-    <collision>
-      <geometry><cylinder radius="0.05" length="0.02"/></geometry>
-    </collision>
   </link>
   <joint name="lidar_to_chassi" type="fixed">

Commit message: Atualização

File: src/camaro_description/urdf/camaro.xacro (robot description, xacro)
@@ -182,5 +182,5 @@
     <parent link="base_link"/>
     <child link="lidarA2"/>
-    <origin xyz="0.42 0 0.25" rpy="0 0 0"/>
+    <origin xyz="0.42 0 0.55" rpy="0 0 0"/>
   </joint>
 </robot>
