Commit message: Atualização mais recente em desenvolvimento (Sem chassi novo) NÂO TESTADO TOTALMENTE

File: src/camaro_description/urdf/camaro.xacro (robot description, xacro)
@@ -12,7 +12,7 @@
     </inertial>
     <visual>
-      <origin xyz="0 0 0.15" rpy="0 0 -3.1416"/>
+      <origin xyz="0 0 0.15" rpy="0 0 0"/>
       <geometry>
-        <mesh filename="file:///home/camaro/camaro_sim_ws/install/camaro_description/share/camaro_description/meshes/camaro_model_final.stl"
+        <mesh filename="file:///home/camaro/camaro_sim_ws/install/camaro_description/share/camaro_description/meshes/camaronovo.glb"
               scale="0.0012 0.0012 0.0012"/>
       </geometry>
@@ -70,20 +70,20 @@
   </joint>
   <!-- ========== RODA DIANTEIRA ESQUERDA ========== -->
-  <link name="front_left_wheel_link">
-    <inertial>
-      <origin rpy="0 0 0" xyz="0 0 0"/>
-      <mass value="1"/>
-      <inertia ixx="0.00303" ixy="0.0" ixz="0.0" iyy="0.00303" iyz="0.0" izz="0.005"/>
-    </inertial>
-    <visual>
-      <origin xyz="0 0 0" rpy="1.5707 0 0"/>
-      <geometry><cylinder radius="0.1" length="0.08"/></geometry>
-      <material name="gray"><color rgba="0.5 0.5 0.5 1"/></material>
-    </visual>
-    <collision>
-      <origin xyz="0 0 0" rpy="1.5707 0 0"/>
-      <geometry><cylinder radius="0.1" length="0.08"/></geometry>
-    </collision>
-  </link>
+<link name="front_left_wheel_link">
+  <inertial>
+    <origin rpy="0 0 0" xyz="0 0 0"/>
+    <mass value="1"/>
+    <inertia ixx="0.00303" ixy="0.0" ixz="0.0" iyy="0.00303" iyz="0.0" izz="0.005"/>
+  </inertial>
+  <visual>
+    <origin xyz="0 0 0" rpy="1.5707 0 0"/>
+    <geometry><cylinder radius="0.1" length="0.08"/></geometry>
+    <material name="gray"><color rgba="0.5 0.5 0.5 1"/></material>
+  </visual>
+  <collision>
+    <origin xyz="0 0 0" rpy="1.5707 0 0"/>
+    <geometry><cylinder radius="0.1" length="0.08"/></geometry>
+  </collision>
+</link>
   <joint name="front_left_wheel_joint" type="revolute">
     <parent link="front_left_wheel_steering_link"/>
@@ -182,5 +182,5 @@
     <parent link="base_link"/>
     <child link="lidarA2"/>
-    <origin xyz="0.42 0 0.55" rpy="0 0 0"/>
+    <origin xyz="0.42 0 0.32" rpy="0 0 0"/>
   </joint>
 </robot>

Commit message: ZED 2i + dashboard: depth_viz, nuvem de pontos, RGB+profundidade, toasts e launcher
- Sensor renomeado para zed2i_rgbd; ponte da nuvem de pontos (/zed/zed_node/points)
- Novo depth_viz_node.py (float32 -> RGB TURBO) no launch + CMakeLists
- web_video_server e rosbridge sobem junto com a simulacao
- Admin: paineis RGB + profundidade lado a lado, botao foto, toasts, polling 4s/30s
- API relativa (/api), status anuncia so os topicos do painel
- abrir_site.py: lançador unico com validacoes

File: src/camaro_description/urdf/camaro.xacro (robot description, xacro)
@@ -32,8 +32,4 @@
       <inertia ixx="0.001" ixy="0.0" ixz="0.0" iyy="0.001" iyz="0.0" izz="0.001"/>
     </inertial>
-    <visual>
-       <geometry><box size="0.05 0.05 0.05"/></geometry>
-       <material name="black"><color rgba="0 0 0 1"/></material>
-    </visual>
     <collision>
       <geometry><box size="0.05 0.05 0.05"/></geometry>
@@ -43,5 +39,5 @@
     <parent link="base_link"/>
     <child link="front_left_wheel_steering_link"/>
-    <origin xyz="0.375 0.23 0.10" rpy="0 0 0"/>
+    <origin xyz="0.375 0.23 0.11" rpy="0 0 0"/>
     <axis xyz="0 0 1"/>
     <limit lower="-0.6" upper="0.6" effort="25" velocity="1.0"/>
@@ -54,8 +50,4 @@
       <inertia ixx="0.001" ixy="0.0" ixz="0.0" iyy="0.001" iyz="0.0" izz="0.001"/>
     </inertial>
-    <visual>
-       <geometry><box size="0.05 0.05 0.05"/></geometry>
-       <material name="black"><color rgba="0 0 0 1"/></material>
-    </visual>
     <collision>
       <geometry><box size="0.05 0.05 0.05"/></geometry>
@@ -65,5 +57,5 @@
     <parent link="base_link"/>
     <child link="front_right_wheel_steering_link"/>
-    <origin xyz="0.375 -0.23 0.10" rpy="0 0 0"/>
+    <origin xyz="0.375 -0.23 0.11" rpy="0 0 0"/>
     <axis xyz="0 0 1"/>
     <limit lower="-0.6" upper="0.6" effort="25" velocity="1.0"/>
@@ -74,14 +66,19 @@
     <origin rpy="0 0 0" xyz="0 0 0"/>
     <mass value="1"/>
-    <inertia ixx="0.00303" ixy="0.0" ixz="0.0" iyy="0.00303" iyz="0.0" izz="0.005"/>
-  </inertial>
-  <visual>
-    <origin xyz="0 0 0" rpy="1.5707 0 0"/>
-    <geometry><cylinder radius="0.1" length="0.08"/></geometry>
-    <material name="gray"><color rgba="0.5 0.5 0.5 1"/></material>
-  </visual>
-  <collision>
-    <origin xyz="0 0 0" rpy="1.5707 0 0"/>
-    <geometry><cylinder radius="0.1" length="0.08"/></geometry>
+    <inertia ixx="0.0036" ixy="0.0" ixz="0.0" iyy="0.0061" iyz="0.0" izz="0.0036"/>
+  </inertial>
+  <visual>
+    <!-- Roda original (rodanova.glb): diâmetro 0.22m (raio 0.11).
+         Eixo da malha é X -> girada para o eixo virar Y (giro -90° p/ esquerda,
+         +90° p/ direita). SEM escala negativa (evita mesh transparente). -->
+    <origin xyz="0 0.0313 0" rpy="0 0 -1.5707"/>
+    <geometry>
+      <mesh filename="package://camaro_description/meshes/rodanova.glb"
+            scale="0.0008462 0.0008462 0.0008462"/>
+    </geometry>
+  </visual>
+  <collision>
+    <origin xyz="0 0 0" rpy="1.5707 0 0"/>
+    <geometry><cylinder radius="0.11" length="0.08"/></geometry>
   </collision>
 </link>
@@ -94,20 +91,23 @@
   </joint>
   <!-- ========== RODA DIANTEIRA DIREITA ========== -->
-  <link name="front_right_wheel_link">
-    <inertial>
-      <origin rpy="0 0 0" xyz="0 0 0"/>
-      <mass value="1"/>
-      <inertia ixx="0.00303" ixy="0.0" ixz="0.0" iyy="0.00303" iyz="0.0" izz="0.005"/>
-    </inertial>
-    <visual>
-      <origin xyz="0 0 0" rpy="1.5707 0 0"/>
-      <geometry><cylinder radius="0.1" length="0.08"/></geometry>
-      <material name="gray"><color rgba="0.5 0.5 0.5 1"/></material>
-    </visual>
-    <collision>
-      <origin xyz="0 0 0" rpy="1.5707 0 0"/>
-      <geometry><cylinder radius="0.1" length="0.08"/></geometry>
-    </collision>
-  </link>
+<link name="front_right_wheel_link">
+  <inertial>
+    <origin rpy="0 0 0" xyz="0 0 0"/>
+    <mass value="1"/>
+    <inertia ixx="0.0036" ixy="0.0" ixz="0.0" iyy="0.0061" iyz="0.0" izz="0.0036"/>
+  </inertial>
+  <visual>
+    <!-- Roda DIREITA aponta p/ fora (-Y) — par espelhado da esquerda. -->
+    <origin xyz="0 -0.0313 0" rpy="0 0 1.5707"/>
+    <geometry>
+      <mesh filename="package://camaro_description/meshes/rodanova.glb"
+            scale="0.0008462 0.0008462 0.0008462"/>
+    </geometry>
+  </visual>
+  <collision>
+    <origin xyz="0 0 0" rpy="1.5707 0 0"/>
+    <geometry><cylinder radius="0.11" length="0.08"/></geometry>
+  </collision>
+</link>
   <joint name="front_right_wheel_joint" type="revolute">
     <parent link="front_right_wheel_steering_link"/>
@@ -118,53 +118,58 @@
   </joint>
   <!-- ========== RODA TRASEIRA ESQUERDA ========== -->
-  <link name="rear_left_wheel_link">
-    <inertial>
-      <origin rpy="0 0 0" xyz="0 0 0"/>
-      <mass value="1"/>
-      <inertia ixx="0.00303" ixy="0.0" ixz="0.0" iyy="0.00303" iyz="0.0" izz="0.005"/>
-    </inertial>
-    <visual>
-      <origin xyz="0 0 0" rpy="1.5707 0 0"/>
-      <geometry><cylinder radius="0.1" length="0.08"/></geometry>
-      <material name="gray"><color rgba="0.5 0.5 0.5 1"/></material>
-    </visual>
-    <collision>
-      <origin xyz="0 0 0" rpy="1.5707 0 0"/>
-      <geometry><cylinder radius="0.1" length="0.08"/></geometry>
-    </collision>
-  </link>
+<link name="rear_left_wheel_link">
+  <inertial>
+    <origin rpy="0 0 0" xyz="0 0 0"/>
+    <mass value="1"/>
+    <inertia ixx="0.0036" ixy="0.0" ixz="0.0" iyy="0.0061" iyz="0.0" izz="0.0036"/>
+  </inertial>
+  <visual>
+    <origin xyz="0 0.0313 0" rpy="0 0 -1.5707"/>
+    <geometry>
+      <mesh filename="package://camaro_description/meshes/rodanova.glb"
+            scale="0.0008462 0.0008462 0.0008462"/>
+    </geometry>
+  </visual>
+  <collision>
+    <origin xyz="0 0 0" rpy="1.5707 0 0"/>
+    <geometry><cylinder radius="0.11" length="0.08"/></geometry>
+  </collision>
+</link>
   <joint name="rear_left_wheel_joint" type="revolute">
     <parent link="base_link"/>
     <child link="rear_left_wheel_link"/>
-    <origin xyz="-0.335 0.23 0.10" rpy="0 0 0"/>
+    <origin xyz="-0.335 0.23 0.11" rpy="0 0 0"/>
     <axis xyz="0 1 0"/>
     <limit lower="-1.79769e+308" upper="1.79769e+308" effort="100" velocity="100"/>
   </joint>
   <!-- ========== RODA TRASEIRA DIREITA ========== -->
-  <link name="rear_right_wheel_link">
-    <inertial>
-      <origin rpy="0 0 0" xyz="0 0 0"/>
-      <mass value="1"/>
-      <inertia ixx="0.00303" ixy="0.0" ixz="0.0" iyy="0.00303" iyz="0.0" izz="0.005"/>
-    </inertial>
-    <visual>
-      <origin xyz="0 0 0" rpy="1.5707 0 0"/>
-      <geometry><cylinder radius="0.1" length="0.08"/></geometry>
-      <material name="gray"><color rgba="0.5 0.5 0.5 1"/></material>
-    </visual>
-    <collision>
-      <origin xyz="0 0 0" rpy="1.5707 0 0"/>
-      <geometry><cylinder radius="0.1" length="0.08"/></geometry>
-    </collision>
-  </link>
+<link name="rear_right_wheel_link">
+  <inertial>
+    <origin rpy="0 0 0" xyz="0 0 0"/>
+    <mass value="1"/>
+    <inertia ixx="0.0036" ixy="0.0" ixz="0.0" iyy="0.0061" iyz="0.0" izz="0.0036"/>
+  </inertial>
+  <visual>
+    <origin xyz="0 -0.0313 0" rpy="0 0 1.5707"/>
+    <geometry>
+      <mesh filename="package://camaro_description/meshes/rodanova.glb"
+            scale="0.0008462 0.0008462 0.0008462"/>
+    </geometry>
+  </visual>
+  <collision>
+    <origin xyz="0 0 0" rpy="1.5707 0 0"/>
+    <geometry><cylinder radius="0.11" length="0.08"/></geometry>
+  </collision>
+</link>
   <joint name="rear_right_wheel_joint" type="revolute">
     <parent link="base_link"/>
     <child link="rear_right_wheel_link"/>
     <!-- JUNTA NEUTRA: Sem rpy aqui! -->
-    <origin xyz="-0.335 -0.23 0.10" rpy="0 0 0"/>
+    <origin xyz="-0.335 -0.23 0.11" rpy="0 0 0"/>
     <axis xyz="0 1 0"/>
     <limit lower="-1.79769e+308" upper="1.79769e+308" effort="100" velocity="100"/>
   </joint>
   <!-- ========== SENSOR LIDAR (CORRIGIDO: SEM COLISÃO) ========== -->
+  <!-- Link do LiDAR SEM visual por enquanto (sensor continua ativo via camaro.gazebo) -->
   <link name="lidarA2">
     <inertial>
@@ -173,13 +178,75 @@
       <inertia ixx="0.001" ixy="0.0" ixz="0.0" iyy="0.001" iyz="0.0" izz="0.001"/>
     </inertial>
-    <visual>
-      <geometry><cylinder radius="0.05" length="0.02"/></geometry>
-      <material name="red"><color rgba="1 0 0 1"/></material>
-    </visual>
   </link>
   <joint name="lidar_to_chassi" type="fixed">
     <parent link="base_link"/>
     <child link="lidarA2"/>
-    <origin xyz="0.52 0 0.50" rpy="0 0 0"/>
+    <!-- LiDAR colado na parte de baixo do chassi, na frente, perto das rodas -->
+    <origin xyz="0.55 0 0.06" rpy="0 0 0"/>
+  </joint>
+  <!-- ========== ZED 2 (VISUAL BÁSICO: suporte + corpo) ========== -->
+  <!-- Visual provisório; depois trocamos pelo mesh real da ZED 2 -->
+  <!-- Haste reduzida apoiada no topo do aerofólio -->
+  <link name="zed_support">
+    <inertial>
+      <origin rpy="0 0 0" xyz="0 0 0.30"/>
+      <mass value="0.05"/>
+      <inertia ixx="0.0001" ixy="0.0" ixz="0.0" iyy="0.0001" iyz="0.0" izz="0.0001"/>
+    </inertial>
+    <visual>
+      <origin rpy="0 0 0" xyz="0 0 0.30"/>
+      <geometry><box size="0.02 0.02 0.60"/></geometry>
+      <material name="preto">
+        <color rgba="0.05 0.05 0.05 1"/>
+      </material>
+    </visual>
+    <visual>
+      <origin rpy="0 0 0" xyz="0 0 0.585"/>
+      <geometry><box size="0.06 0.06 0.03"/></geometry>
+      <material name="preto">
+        <color rgba="0.05 0.05 0.05 1"/>
+      </material>
+    </visual>
+    <collision>
+      <origin rpy="0 0 0" xyz="0 0 0.30"/>
+      <geometry><box size="0.02 0.02 0.60"/></geometry>
+    </collision>
+  </link>
+  <joint name="zed_support_joint" type="fixed">
+    <parent link="base_link"/>
+    <child link="zed_support"/>
+    <origin xyz="-0.58 0 0.25" rpy="0 0 0"/>
+  </joint>
+  <link name="zed_mount">
+    <inertial>
+      <origin rpy="0 0 0" xyz="0 0 0.015"/>
+      <mass value="0.08"/>
+      <inertia ixx="0.0005" ixy="0.0" ixz="0.0" iyy="0.0005" iyz="0.0" izz="0.0005"/>
+    </inertial>
+    <visual>
+      <origin rpy="0 0 -1.5708" xyz="0 0 0.0018"/>
+      <geometry>
+        <mesh filename="package://camaro_description/meshes/zed2_detailed.stl"/>
+      </geometry>
+      <material name="zed_body">
+        <color rgba="0.18 0.18 0.18 1"/>
+      </material>
+    </visual>
+    <collision>
+      <origin rpy="0 0 0" xyz="0 0 0.015"/>
+      <geometry><box size="0.035 0.18 0.035"/></geometry>
+    </collision>
+  </link>
+  <joint name="zed_mount_joint" type="fixed">
+    <parent link="zed_support"/>
+    <child link="zed_mount"/>
+    <origin xyz="0 0 0.60" rpy="0 0 0"/>
+  </joint>
+  <!-- Câmera do usuário (2D), virada para trás, sobre a ZED -->
+  <link name="camera_user_link"/>
+  <joint name="camera_user_joint" type="fixed">
+    <parent link="zed_mount"/>
+    <child link="camera_user_link"/>
+    <origin xyz="0 0 0.03" rpy="0 0 3.14159"/>
   </joint>
 </robot>
